File: samples/macropad-buggy/macropad-buggy.kicad_pcb (KiCad board)
At the start: 2 copper layers, 87 x 58 mm, 22 parts, among them J1 Battery, SW1 SW_Push, SW10 Power, SW2 SW_Push, SW3 SW_Push, SW4 SW_Push, SW5 SW_Push, SW6 SW_Push, SW7 SW_Push, SW8 SW_Push, SW9 SW_Push, U1 nice!nano

Commit message: Rename to fabready, add Settings tab for fabready.json, split docs
- Rename pcbcheck to fabready across crates, binaries, app, config file and output folder
- Desktop app: Settings tab that edits the project's fabready.json, and a Waive button on findings
- The header profile picker saves to fabready.json, so the app, CLI and agents agree
- Validate config on load and save (an invalid keyboard pattern used to crash checks)
- Shorter README; details moved to docs/ and AGENTS.md
Parts:
- J1: footprint pcbcheck_samples:JST_PH_2pin -> fabready_samples:JST_PH_2pin
- SW1, SW2, SW3, SW4, SW5, SW6, SW7, SW8, SW9: footprint pcbcheck_samples:SW_MX_1u -> fabready_samples:SW_MX_1u
- SW10: footprint pcbcheck_samples:SW_Slide_SPDT -> fabready_samples:SW_Slide_SPDT
- U1: footprint pcbcheck_samples:nice_nano -> fabready_samples:nice_nano
Changed lines of the file:
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@@
-(kicad_pcb (version 20240108) (generator "pcbcheck_sample") (generator_version "8.0")
+(kicad_pcb (version 20240108) (generator "fabready_sample") (generator_version "8.0")
   (general (thickness 1.6) (legacy_teardrops no))
   (paper "A4")
@@
   (net 17 "BAT+")
   (gr_rect (start 100 100) (end 187 158) (stroke (width 0.1) (type default)) (fill none) (layer "Edge.Cuts"))
-  (footprint "pcbcheck_samples:nice_nano" (layer "F.Cu") (at 175.000 118.000)
+  (footprint "fabready_samples:nice_nano" (layer "F.Cu") (at 175.000 118.000)
     (property "Reference" "U1" (at 0 -17.50 0) (layer "F.SilkS") (effects (font (size 1 1) (thickness 0.15))))
     (property "Value" "nice!nano" (at 0 17.50 0) (layer "F.Fab") (effects (font (size 1 1) (thickness 0.15))))
@@
     (pad "13" thru_hole circle (at 7.62 13.97) (size 1.7 1.7) (drill 1.0) (layers "*.Cu" "*.Mask") (pinfunction "B6") (pintype "passive"))
   )
-  (footprint "pcbcheck_samples:SW_MX_1u" (layer "F.Cu") (at 110.000 110.000)
+  (footprint "fabready_samples:SW_MX_1u" (layer "F.Cu") (at 110.000 110.000)
     (property "Reference" "SW1" (at 0 -8.00 0) (layer "F.SilkS") (effects (font (size 1 1) (thickness 0.15))))
     (property "Value" "SW_Push" (at 0 8.00 0) (layer "F.Fab") (effects (font (size 1 1) (thickness 0.15))))
@@
   )
   (segment (start 108.350 115.000) (end 108.350 117.000) (width 0.25) (layer "B.Cu") (net 4 "ROW0"))
-  (footprint "pcbcheck_samples:SW_MX_1u" (layer "F.Cu") (at 129.050 110.000)
+  (footprint "fabready_samples:SW_MX_1u" (layer "F.Cu") (at 129.050 110.000)
     (property "Reference" "SW2" (at 0 -8.00 0) (layer "F.SilkS") (effects (font (size 1 1) (thickness 0.15))))
     (property "Value" "SW_Push" (at 0 8.00 0) (layer "F.Fab") (effects (font (size 1 1) (thickness 0.15))))
@@
   )
   (segment (start 127.400 115.000) (end 127.400 117.000) (width 0.25) (layer "B.Cu") (net 4 "ROW0"))
-  (footprint "pcbcheck_samples:SW_MX_1u" (layer "F.Cu") (at 148.100 110.000)
+  (footprint "fabready_samples:SW_MX_1u" (layer "F.Cu") (at 148.100 110.000)
     (property "Reference" "SW3" (at 0 -8.00 0) (layer "F.SilkS") (effects (font (size 1 1) (thickness 0.15))))
     (property "Value" "SW_Push" (at 0 8.00 0) (layer "F.Fab") (effects (font (size 1 1) (thickness 0.15))))
@@
   )
   (segment (start 146.450 115.000) (end 146.450 117.000) (width 0.25) (layer "B.Cu") (net 4 "ROW0"))
-  (footprint "pcbcheck_samples:SW_MX_1u" (layer "F.Cu") (at 110.000 129.050)
+  (footprint "fabready_samples:SW_MX_1u" (layer "F.Cu") (at 110.000 129.050)
     (property "Reference" "SW4" (at 0 -8.00 0) (layer "F.SilkS") (effects (font (size 1 1) (thickness 0.15))))
     (property "Value" "SW_Push" (at 0 8.00 0) (layer "F.Fab") (effects (font (size 1 1) (thickness 0.15))))
@@
   )
   (segment (start 108.350 134.050) (end 108.350 136.050) (width 0.25) (layer "B.Cu") (net 5 "ROW1"))
-  (footprint "pcbcheck_samples:SW_MX_1u" (layer "F.Cu") (at 129.050 129.050)
+  (footprint "fabready_samples:SW_MX_1u" (layer "F.Cu") (at 129.050 129.050)
     (property "Reference" "SW5" (at 0 -8.00 0) (layer "F.SilkS") (effects (font (size 1 1) (thickness 0.15))))
     (property "Value" "SW_Push" (at 0 8.00 0) (layer "F.Fab") (effects (font (size 1 1) (thickness 0.15))))
@@
   )
   (segment (start 127.400 134.050) (end 127.400 136.050) (width 0.25) (layer "B.Cu") (net 5 "ROW1"))
-  (footprint "pcbcheck_samples:SW_MX_1u" (layer "F.Cu") (at 148.100 129.050)
+  (footprint "fabready_samples:SW_MX_1u" (layer "F.Cu") (at 148.100 129.050)
     (property "Reference" "SW6" (at 0 -8.00 0) (layer "F.SilkS") (effects (font (size 1 1) (thickness 0.15))))
     (property "Value" "SW_Push" (at 0 8.00 0) (layer "F.Fab") (effects (font (size 1 1) (thickness 0.15))))
@@
   )
   (segment (start 146.450 134.050) (end 146.450 136.050) (width 0.25) (layer "B.Cu") (net 5 "ROW1"))
-  (footprint "pcbcheck_samples:SW_MX_1u" (layer "F.Cu") (at 110.000 148.100)
+  (footprint "fabready_samples:SW_MX_1u" (layer "F.Cu") (at 110.000 148.100)
     (property "Reference" "SW7" (at 0 -8.00 0) (layer "F.SilkS") (effects (font (size 1 1) (thickness 0.15))))
     (property "Value" "SW_Push" (at 0 8.00 0) (layer "F.Fab") (effects (font (size 1 1) (thickness 0.15))))
@@
   )
   (segment (start 108.350 153.100) (end 108.350 155.100) (width 0.25) (layer "B.Cu") (net 6 "ROW2"))
-  (footprint "pcbcheck_samples:SW_MX_1u" (layer "F.Cu") (at 129.050 148.100)
+  (footprint "fabready_samples:SW_MX_1u" (layer "F.Cu") (at 129.050 148.100)
     (property "Reference" "SW8" (at 0 -8.00 0) (layer "F.SilkS") (effects (font (size 1 1) (thickness 0.15))))
     (property "Value" "SW_Push" (at 0 8.00 0) (layer "F.Fab") (effects (font (size 1 1) (thickness 0.15))))
@@
   )
   (segment (start 127.400 153.100) (end 127.400 155.100) (width 0.25) (layer "B.Cu") (net 6 "ROW2"))
-  (footprint "pcbcheck_samples:SW_MX_1u" (layer "F.Cu") (at 148.100 148.100)
+  (footprint "fabready_samples:SW_MX_1u" (layer "F.Cu") (at 148.100 148.100)
     (property "Reference" "SW9" (at 0 -8.00 0) (layer "F.SilkS") (effects (font (size 1 1) (thickness 0.15))))
     (property "Value" "SW_Push" (at 0 8.00 0) (layer "F.Fab") (effects (font (size 1 1) (thickness 0.15))))
@@
   (segment (start 163.300 116.730) (end 167.380 116.730) (width 0.25) (layer "F.Cu") (net 3 "COL1"))
   (segment (start 144.290 107.460) (end 144.290 145.560) (width 0.25) (layer "F.Cu") (net 10 "COL2"))
-  (footprint "pcbcheck_samples:JST_PH_2pin" (layer "F.Cu") (at 176.000 150.000)
+  (footprint "fabready_samples:JST_PH_2pin" (layer "F.Cu") (at 176.000 150.000)
     (property "Reference" "J1" (at 0 -3.50 0) (layer "F.SilkS") (effects (font (size 1 1) (thickness 0.15))))
     (property "Value" "Battery" (at 0 3.50 0) (layer "F.Fab") (effects (font (size 1 1) (thickness 0.15))))
@@
     (pad "2" thru_hole circle (at 1 0) (size 1.4 1.4) (drill 0.8) (layers "*.Cu" "*.Mask") (net 1 "GND") (pinfunction "-") (pintype "passive"))
   )
-  (footprint "pcbcheck_samples:SW_Slide_SPDT" (layer "F.Cu") (at 176.000 142.000)
+  (footprint "fabready_samples:SW_Slide_SPDT" (layer "F.Cu") (at 176.000 142.000)
     (property "Reference" "SW10" (at 0 -2.50 0) (layer "F.SilkS") (effects (font (size 1 1) (thickness 0.15))))
     (property "Value" "Power" (at 0 2.50 0) (layer "F.Fab") (effects (font (size 1 1) (thickness 0.15))))
